Commit message: Porting velocity controllers and imu

File: urdf/ezrassor.xacro (robot description, xacro)
@@ -1,212 +1,200 @@
 <?xml version='1.0'?>
-<robot name="ezrassor" xmlns:xacro="http://www.ros.org/wiki/xacro">
-  <xacro:property name="cameraSize" value="0.01"/>
-  <xacro:property name="cameraMass" value="0.1"/>
-  <xacro:include filename="$(find ezrassor_sim_description)/urdf/ezrassor.gazebo" />
-  <xacro:include filename="$(find ezrassor_sim_description)/urdf/materials.xacro" />
-  <xacro:include filename="$(find ezrassor_sim_description)/urdf/macros.xacro" />
-  <!--Below are all of the robot's Links/-->
-  <link name='base_link'>
-   <pose>0 0 0 0 0 0</pose>
-  </link>
-  <link name='body'>
-    <pose>0 0 0 0 0 0</pose>
-    <inertial>
-      <mass value="15.0"/>
-      <origin xyz="0 0 0" rpy=" 0 0 0"/>
-      <inertia
-          ixx="0.5" ixy="0" ixz="0"
-          iyy="1.0" iyz="0"
-          izz="0.1"
-      />
-    </inertial>
-    <collision name='collision'>
-      <origin xyz="0 0 0" rpy=" 0 0 0"/>
-      <geometry>
-        <base_unit/>
-      </geometry>
-    </collision>
-    <visual name='base_link_visual'>
-      <origin xyz="0 0 0" rpy=" 0 0 0"/>
-      <geometry>
-        <base_unit/>
-      </geometry>
-    </visual>
-  </link>
-  <link name="left_wheel_front">
-    <collision name="collision">
-      <origin xyz="0 0 0" rpy="0 0 0"/>
-      <geometry>
-        <robot_wheel />
-      </geometry>
-      <surface>
-        <friction>
-          <mu> .6 </mu>
-          <mu2> .6 </mu2>
-        </friction>
-      </surface>
-      <surface>
-        <friction>
-          <mu> .6 </mu>
-          <mu2> .6 </mu2>
-        </friction>
-      </surface>
-    </collision>
-    <visual name="left_wheel_front_visual">
-      <origin xyz="0 0 0" rpy="0 0 0"/>
-      <geometry>
-        <robot_wheel />
-      </geometry>
-    </visual>
-    <inertial>
-      <origin xyz="0 0 0" rpy="0 0 0" />
-      <mass value="5"/>
-      <cylinder_inertia m="5" r="0.18" h="0.2"/>
-    </inertial>
-  </link>
-  <link name="right_wheel_front">
-    <collision name="collision">
-      <origin xyz="0 0 0" rpy="0 0 3.14159"/>
-      <geometry>
-        <robot_wheel />
-      </geometry>
-      <surface>
-        <friction>
-        <mu> .6 </mu>
-        <mu2> .6 </mu2>
-        </friction>
-      </surface>
-    </collision>
-    <visual name="right_wheel_front_visual">
-      <origin xyz="0 0 0" rpy="0 0 3.14159"/>
-      <geometry>
-        <robot_wheel />
-      </geometry>
-    </visual>
-    <inertial>
-      <origin xyz="0 0 0" rpy="0 0 3.14159"/>
-      <mass value="5"/>
-      <cylinder_inertia m="5" r="0.18" h="0.2"/>
-    </inertial>
-  </link>
-  <link name="left_wheel_back">
-    <collision name="collision">
-      <origin xyz="0 0 0" rpy="0 0 0"/>
-      <geometry>
-        <robot_wheel />
-      </geometry>
-        <surface>
-          <friction>
-            <mu> .6 </mu>
-            <mu2> .6 </mu2>
-         </friction>
-        </surface>
-    </collision>
-    <visual name="left_wheel_back_visual">
-      <origin xyz="0 0 0" rpy="0 0 0"/>
-      <geometry>
-        <robot_wheel />
-      </geometry>
-    </visual>
-    <inertial>
-      <origin xyz="0 0 0" rpy="0 0 0"/>
-      <mass value="5"/>
-      <cylinder_inertia m="5" r="0.18" h="0.2"/>
-    </inertial>
-  </link>
-  <link name="right_wheel_back">
-    <collision name="collision">
-      <origin xyz="0 0 0" rpy="0 0 3.14159"/>
-      <geometry>
-        <robot_wheel />
-      </geometry>
-      <surface>
-        <friction>
-          <mu> .6 </mu>
-          <mu2> .6 </mu2>
-        </friction>
-      </surface>
-    </collision>
-    <visual name="right_wheel_back_visual">
-      <origin xyz="0 0 0" rpy="0 0 3.14159"/>
-      <geometry>
-        <robot_wheel />
-      </geometry>
-    </visual>
-    <inertial>
-      <origin xyz="0 0 0" rpy="0 0 3.14159"/>
-      <mass value="5"/>
-      <cylinder_inertia m="5" r="0.18" h="0.2"/>
-    </inertial>
-  </link>
-  <link name="arm_front">
-    <collision name="collision">
-      <origin xyz="0 0 0" rpy="0 0 0"/>
-      <geometry>
-        <drum_arm />
-      </geometry>
-    </collision>
-    <visual name="visual">
-      <origin xyz="0 0 0" rpy="0 0 0" />
-      <geometry>
-        <drum_arm />
-      </geometry>
-    </visual>
-    <inertial>
-      <origin xyz="0 0 0" rpy="0 0 0"/>
-      <mass value="5"/>
-      <cylinder_inertia m="5" r="0.05" h="0.3"/>
-    </inertial>
-  </link>
-  <link name="arm_back">
-    <collision name="collision">
-      <origin xyz="0 0 0" rpy="3.1415 0 3.1415"/>
-      <geometry>
-        <drum_arm />
-      </geometry>
-    </collision>
-    <visual name="visual">
-      <origin xyz="0 0 0" rpy="3.1415 0 3.1415"/>
-      <geometry>
-        <drum_arm />
-      </geometry>
-    </visual>
-    <inertial>
-      <origin xyz="0 0 0" rpy="0 0 3.1415"/>
-      <mass value="5"/>
-      <cylinder_inertia m="5" r="0.05" h="0.3"/>
-      <inertia
-        ixx="1.0" ixy="0.0" ixz="0.0"
-        iyy="1.0" iyz="0.0"
-        izz="1.0"/>
-    </inertial>
-  </link>
-  <link name="drum_front">
-    <!-- <collision name="collision">
-      <origin xyz="0 0 0" rpy="0 0 0"/>
-      <geometry>
-        <robot_arm_drum />
-      </geometry>
-    </collision>-->
-    <collision name="collision">
-      <origin xyz="0 0 0" rpy="0 1.5707 1.5707"/>
-      <geometry>
-        <cylinder radius="0.1839" length="1.0"/>
-      </geometry>
-    </collision>
-    <visual name="drum_front_visual">
-      <origin xyz="0 0 0" rpy="0 0 0"/>
-      <geometry>
-        <robot_arm_drum />
-      </geometry>
-    </visual>
-    <inertial>
-      <origin xyz="0 0 0" rpy="0 0 0"/>
-      <mass value="5"/>
-      <cylinder_inertia m="5" r="0.1839" h="1.0"/>
-    </inertial>
-  </link>
-  <link name="drum_back">
-    <!-- <collision name="collision">
+<robot name="ezrassor"
+    xmlns:xacro="http://www.ros.org/wiki/xacro">
+    <xacro:property name="cameraSize" value="0.01"/>
+    <xacro:property name="cameraMass" value="0.1"/>
+    <xacro:include filename="$(find ezrassor_sim_description)/urdf/ezrassor.gazebo" />
+    <xacro:include filename="$(find ezrassor_sim_description)/urdf/materials.xacro" />
+    <xacro:include filename="$(find ezrassor_sim_description)/urdf/macros.xacro" />
+    <!--Below are all of the robot's Links/-->
+    <link name='base_link'>
+        <pose>0 0 0 0 0 0</pose>
+    </link>
+    <link name='body'>
+        <pose>0 0 0 0 0 0</pose>
+        <inertial>
+            <mass value="15.0"/>
+            <origin xyz="0 0 0" rpy=" 0 0 0"/>
+            <inertia ixx="0.5" ixy="0" ixz="0" iyy="1.0" iyz="0" izz="0.1" />
+        </inertial>
+        <collision name='collision'>
+            <origin xyz="0 0 0" rpy=" 0 0 0"/>
+            <geometry>
+                <xacro:base_unit/>
+            </geometry>
+        </collision>
+        <visual name='base_link_visual'>
+            <origin xyz="0 0 0" rpy=" 0 0 0"/>
+            <geometry>
+                <xacro:base_unit/>
+            </geometry>
+        </visual>
+    </link>
+    <link name="left_wheel_front">
+        <collision name="collision">
+            <origin xyz="0 0 0" rpy="0 0 0"/>
+            <geometry>
+                <xacro:robot_wheel />
+            </geometry>
+            <surface>
+                <friction>
+                    <mu> .6 </mu>
+                    <mu2> .6 </mu2>
+                </friction>
+            </surface>
+            <surface>
+                <friction>
+                    <mu> .6 </mu>
+                    <mu2> .6 </mu2>
+                </friction>
+            </surface>
+        </collision>
+        <visual name="left_wheel_front_visual">
+            <origin xyz="0 0 0" rpy="0 0 0"/>
+            <geometry>
+                <xacro:robot_wheel />
+            </geometry>
+        </visual>
+        <inertial>
+            <origin xyz="0 0 0" rpy="0 0 0" />
+            <mass value="5"/>
+            <xacro:cylinder_inertia m="5" r="0.18" h="0.2"/>
+        </inertial>
+    </link>
+    <link name="right_wheel_front">
+        <collision name="collision">
+            <origin xyz="0 0 0" rpy="0 0 3.14159"/>
+            <geometry>
+                <xacro:robot_wheel />
+            </geometry>
+            <surface>
+                <friction>
+                    <mu> .6 </mu>
+                    <mu2> .6 </mu2>
+                </friction>
+            </surface>
+        </collision>
+        <visual name="right_wheel_front_visual">
+            <origin xyz="0 0 0" rpy="0 0 3.14159"/>
+            <geometry>
+                <xacro:robot_wheel />
+            </geometry>
+        </visual>
+        <inertial>
+            <origin xyz="0 0 0" rpy="0 0 3.14159"/>
+            <mass value="5"/>
+            <xacro:cylinder_inertia m="5" r="0.18" h="0.2"/>
+        </inertial>
+    </link>
+    <link name="left_wheel_back">
+        <collision name="collision">
+            <origin xyz="0 0 0" rpy="0 0 0"/>
+            <geometry>
+                <xacro:robot_wheel />
+            </geometry>
+            <surface>
+                <friction>
+                    <mu> .6 </mu>
+                    <mu2> .6 </mu2>
+                </friction>
+            </surface>
+        </collision>
+        <visual name="left_wheel_back_visual">
+            <origin xyz="0 0 0" rpy="0 0 0"/>
+            <geometry>
+                <xacro:robot_wheel />
+            </geometry>
+        </visual>
+        <inertial>
+            <origin xyz="0 0 0" rpy="0 0 0"/>
+            <mass value="5"/>
+            <xacro:cylinder_inertia m="5" r="0.18" h="0.2"/>
+        </inertial>
+    </link>
+    <link name="right_wheel_back">
+        <collision name="collision">
+            <origin xyz="0 0 0" rpy="0 0 3.14159"/>
+            <geometry>
+                <xacro:robot_wheel />
+            </geometry>
+            <surface>
+                <friction>
+                    <mu> .6 </mu>
+                    <mu2> .6 </mu2>
+                </friction>
+            </surface>
+        </collision>
+        <visual name="right_wheel_back_visual">
+            <origin xyz="0 0 0" rpy="0 0 3.14159"/>
+            <geometry>
+                <xacro:robot_wheel />
+            </geometry>
+        </visual>
+        <inertial>
+            <origin xyz="0 0 0" rpy="0 0 3.14159"/>
+            <mass value="5"/>
+            <xacro:cylinder_inertia m="5" r="0.18" h="0.2"/>
+        </inertial>
+    </link>
+    <link name="arm_front">
+        <collision name="collision">
+            <origin xyz="0 0 0" rpy="0 0 0"/>
+            <geometry>
+                <xacro:drum_arm />
+            </geometry>
+        </collision>
+        <visual name="visual">
+            <origin xyz="0 0 0" rpy="0 0 0" />
+            <geometry>
+                <xacro:drum_arm />
+            </geometry>
+        </visual>
+        <inertial>
+            <origin xyz="0 0 0" rpy="0 0 0"/>
+            <mass value="5"/>
+            <xacro:cylinder_inertia m="5" r="0.05" h="0.3"/>
+        </inertial>
+    </link>
+    <link name="arm_back">
+        <collision name="collision">
+            <origin xyz="0 0 0" rpy="3.1415 0 3.1415"/>
+            <geometry>
+                <xacro:drum_arm />
+            </geometry>
+        </collision>
+        <visual name="visual">
+            <origin xyz="0 0 0" rpy="3.1415 0 3.1415"/>
+            <geometry>
+                <xacro:drum_arm />
+            </geometry>
+        </visual>
+        <inertial>
+            <origin xyz="0 0 0" rpy="0 0 3.1415"/>
+            <mass value="5"/>
+            <xacro:cylinder_inertia m="5" r="0.05" h="0.3"/>
+            <inertia ixx="1.0" ixy="0.0" ixz="0.0" iyy="1.0" iyz="0.0" izz="1.0"/>
+        </inertial>
+    </link>
+    <link name="drum_front">
+        <collision name="collision">
+            <origin xyz="0 0 0" rpy="0 1.5707 1.5707"/>
+            <geometry>
+                <cylinder radius="0.1839" length="1.0"/>
+            </geometry>
+        </collision>
+        <visual name="drum_front_visual">
+            <origin xyz="0 0 0" rpy="0 0 0"/>
+            <geometry>
+                <xacro:robot_arm_drum />
+            </geometry>
+        </visual>
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
File: urdf/macros.xacro (robot description, xacro)
@@ -37,17 +37,17 @@
     <!-- VISUAL AND COLLISION MACROS -->
     <xacro:macro name="robot_arm">
-        <mesh filename="package://ezrassor_sim_description/meshes/drum_arm_short.dae" scale="1.0 1.0 1.0"></mesh>
+        <mesh filename="file://$(find ezrassor_sim_description)/meshes/drum_arm_short.dae" scale="1.0 1.0 1.0"></mesh>
     </xacro:macro>
     <xacro:macro name="robot_arm_drum">
-        <mesh filename="package://ezrassor_sim_description/meshes/drum.dae" scale="0.35 0.35 0.35"></mesh>
+        <mesh filename="file://$(find ezrassor_sim_description)/meshes/drum.dae" scale="0.35 0.35 0.35"></mesh>
     </xacro:macro>
     <xacro:macro name="robot_wheel">
-        <mesh filename="package://ezrassor_sim_description/meshes/wheel.dae" scale="0.35 0.35 0.35"></mesh>
+        <mesh filename="file://$(find ezrassor_sim_description)/meshes/wheel.dae" scale="0.35 0.35 0.35"></mesh>
     </xacro:macro>
     <xacro:macro name="base_unit">
-        <mesh filename="package://ezrassor_sim_description/meshes/base_unit.dae" scale="0.35 0.35 0.35"></mesh>
+        <mesh filename="file://$(find ezrassor_sim_description)/meshes/base_unit.dae" scale="0.35 0.35 0.35"></mesh>
     </xacro:macro>
     <xacro:macro name="drum_arm">
-        <mesh filename="package://ezrassor_sim_description/meshes/drum_arm.dae" scale="0.35 0.35 0.35"></mesh>
+        <mesh filename="file://$(find ezrassor_sim_description)/meshes/drum_arm.dae" scale="0.35 0.35 0.35"></mesh>
     </xacro:macro>
 </robot>

Commit message: multiple robots can now be spawned from ros2

File: urdf/ezrassor.xacro (robot description, xacro)
@@ -4,8 +4,9 @@
     <xacro:property name="cameraSize" value="0.01"/>
     <xacro:property name="cameraMass" value="0.1"/>
+    <!--Gazebo included file contains plugins and plugin values-->
     <xacro:include filename="$(find ezrassor_sim_description)/urdf/ezrassor.gazebo" />
     <xacro:include filename="$(find ezrassor_sim_description)/urdf/materials.xacro" />
     <xacro:include filename="$(find ezrassor_sim_description)/urdf/macros.xacro" />
-    <!--Below are all of the robot's Links/-->
+    <!--Tags below represent robot links and joints only-->
     <link name='base_link'>
         <pose>0 0 0 0 0 0</pose>
@@ -196,10 +197,4 @@
     </link>
     <link name="drum_back">
-        <!-- <collision name="collision">
-      <origin xyz="0 0 0" rpy="0 0 3.14159"/>
-      <geometry>
-        <robot_arm_drum />
-      </geometry>
-    </collision> -->
         <collision name="collision">
             <origin xyz="0 0 0" rpy="0 1.5707 1.5707"/>
@@ -351,49 +346,3 @@
         <joint_properties damping="0.0" friction="0.0"/>
     </joint>
-    <ros2_control name="GazeboSystem" type="system">
-        <hardware>
-            <plugin>gazebo_ros2_control/GazeboSystem</plugin>
-        </hardware>
-        <joint name="left_wheel_front_hinge">
-            <command_interface name="velocity">
-                <param name="min">-10</param>
-                <param name="max">10</param>
-            </command_interface>
-            <state_interface name="position" />
-            <state_interface name="velocity" />
-            <state_interface name="effort" />
-        </joint>
-        <joint name="right_wheel_front_hinge">
-            <command_interface name="velocity">
-                <param name="min">-10</param>
-                <param name="max">10</param>
-            </command_interface>
-            <state_interface name="position" />
-            <state_interface name="velocity" />
-            <state_interface name="effort" />
-        </joint>
-        <joint name="left_wheel_back_hinge">
-            <command_interface name="velocity">
-                <param name="min">-10</param>
-                <param name="max">10</param>
-            </command_interface>
-            <state_interface name="position" />
-            <state_interface name="velocity" />
-            <state_interface name="effort" />
-        </joint>
-        <joint name="right_wheel_back_hinge">
-            <command_interface name="velocity">
-                <param name="min">-10</param>
-                <param name="max">10</param>
-            </command_interface>
-            <state_interface name="position" />
-            <state_interface name="velocity" />
-            <state_interface name="effort" />
-        </joint>
-    </ros2_control>
-    <gazebo>
-        <plugin filename="libgazebo_ros2_control.so" name="gazebo_ros2_control">
-            <parameters>$(find ezrassor_sim_description)/config/controllers.yaml</parameters>
-        </plugin>
-    </gazebo>
 </robot>

File: urdf/macros.xacro (robot description, xacro)
@@ -1,34 +1,23 @@
 <?xml version='1.0'?>
-<robot name="ezrassor" xmlns:xacro="http://www.ros.org/wiki/xacro">
+<robot name="ezrassor"
+    xmlns:xacro="http://www.ros.org/wiki/xacro">
     <!-- Inertia Tensors Used: https://en.wikipedia.org/wiki/List_of_moments_of_inertia#List_of_3D_inertia_tensors -->
     <xacro:macro name="cylinder_inertia" params="m r h">
-    <inertia
-        ixx="${m*((3*r*r)+(h*h))/12}" ixy = "0"                 ixz = "0"
-                                  iyy="${m*((3*r*r)+(h*h))/12}" iyz = "0"
-                                                            izz="${(m*(r*r))/2}"
-    />
+        <inertia ixx="${m*((3*r*r)+(h*h))/12}" ixy = "0"                 ixz = "0" iyy="${m*((3*r*r)+(h*h))/12}" iyz = "0" izz="${(m*(r*r))/2}" />
     </xacro:macro>
     <xacro:macro name="box_inertia" params="m x y z">
-    <inertia  ixx="${m*(y*y+z*z)/12}" ixy = "0" ixz = "0"
-        iyy="${m*(x*x+z*z)/12}" iyz = "0"
-        izz="${m*(x*x+z*z)/12}"
-    />
+        <inertia ixx="${m*(y*y+z*z)/12}" ixy = "0" ixz = "0" iyy="${m*(x*x+z*z)/12}" iyz = "0" izz="${m*(x*x+z*z)/12}" />
     </xacro:macro>
     <xacro:macro name="sphere_inertia" params="m r">
-    <inertia  ixx="${2*m*r*r/5}" ixy = "0" ixz = "0"
-        iyy="${2*m*r*r/5}" iyz = "0"
-        izz="${2*m*r*r/5}"
-    />
+        <inertia ixx="${2*m*r*r/5}" ixy = "0" ixz = "0" iyy="${2*m*r*r/5}" iyz = "0" izz="${2*m*r*r/5}" />
     </xacro:macro>
     <xacro:macro name="slender_rod_along_y_inertia" params="m l mass_about">
         <xacro:if value="${mass_about == 'end'}">
-            <inertia
-                ixx="${1/3*m*(l*l)}" ixy = "0"
+            <inertia ixx="${1/3*m*(l*l)}" ixy = "0"
                 ixz = "0" iyy="0"
                 iyz = "0" izz="${1/3*m*(l*l)}" />
         </xacro:if>
         <xacro:unless value="${mass_about == 'center'}">
-            <inertia
-                ixx="${1/12*m*(l*l)}" ixy = "0"
+            <inertia ixx="${1/12*m*(l*l)}" ixy = "0"
                 ixz = "0" iyy="0"
                 iyz = "0" izz="${1/12*m*(l*l)}" />

File: urdf/materials.xacro (robot description, xacro)
@@ -1,27 +1,28 @@
 <?xml version='1.0'?>
-<robot name="ezrassor" xmlns:xacro="http://www.ros.org/wiki/xacro">
-  <material name="black">
-    <color rgba="0.0 0.0 0.0 1.0"/>
-  </material>
-  <material name="blue">
-    <color rgba="0.0 0.0 0.8 1.0"/>
-  </material>
-  <material name="green">
-    <color rgba="0.0 0.8 0.0 1.0"/>
-  </material>
-  <material name="grey">
-    <color rgba="0.2 0.2 0.2 1.0"/>
-  </material>
-  <material name="orange">
-    <color rgba="${255/255} ${108/255} ${10/255} 1.0"/>
-  </material>
-  <material name="brown">
-    <color rgba="${222/255} ${207/255} ${195/255} 1.0"/>
-  </material>
-  <material name="red">
-    <color rgba="0.8 0.0 0.0 1.0"/>
-  </material>
-  <material name="white">
-    <color rgba="1.0 1.0 1.0 1.0"/>
-  </material>
+<robot name="ezrassor"
+    xmlns:xacro="http://www.ros.org/wiki/xacro">
+    <material name="black">
+        <color rgba="0.0 0.0 0.0 1.0"/>
+    </material>
+    <material name="blue">
+        <color rgba="0.0 0.0 0.8 1.0"/>
+    </material>
+    <material name="green">
+        <color rgba="0.0 0.8 0.0 1.0"/>
+    </material>
+    <material name="grey">
+        <color rgba="0.2 0.2 0.2 1.0"/>
+    </material>
+    <material name="orange">
+        <color rgba="${255/255} ${108/255} ${10/255} 1.0"/>
+    </material>
+    <material name="brown">
+        <color rgba="${222/255} ${207/255} ${195/255} 1.0"/>
+    </material>
+    <material name="red">
+        <color rgba="0.8 0.0 0.0 1.0"/>
+    </material>
+    <material name="white">
+        <color rgba="1.0 1.0 1.0 1.0"/>
+    </material>
 </robot>
