Commit message: Simplifying xacro structure and updating the controller manager

File: urdf/macros.xacro (robot description, xacro)
@@ -24,19 +24,6 @@
         </xacro:unless>
     </xacro:macro>
-    <!-- VISUAL AND COLLISION MACROS -->
-    <xacro:macro name="robot_arm">
-        <mesh filename="file://$(find ezrassor_sim_description)/meshes/drum_arm_short.dae" scale="1.0 1.0 1.0"></mesh>
-    </xacro:macro>
-    <xacro:macro name="robot_arm_drum">
-        <mesh filename="file://$(find ezrassor_sim_description)/meshes/drum.dae" scale="0.35 0.35 0.35"></mesh>
-    </xacro:macro>
-    <xacro:macro name="robot_wheel">
-        <mesh filename="file://$(find ezrassor_sim_description)/meshes/wheel.dae" scale="0.35 0.35 0.35"></mesh>
-    </xacro:macro>
     <xacro:macro name="base_unit">
         <mesh filename="file://$(find ezrassor_sim_description)/meshes/base_unit.dae" scale="0.35 0.35 0.35"></mesh>
     </xacro:macro>
-    <xacro:macro name="drum_arm">
-        <mesh filename="file://$(find ezrassor_sim_description)/meshes/drum_arm.dae" scale="0.35 0.35 0.35"></mesh>
-    </xacro:macro>
 </robot>

Commit message: ROS2 Foxy - ROS1 control+description port (#3)
* Porting velocity controllers and imu

* Adding lint workflow and documentation

* Updating testing lines in doc

* Creating sim driver nodes for the arms, wheels, and drums

* Updating blender models

* Simplifying xacro structure and updating the controller manager

File: urdf/macros.xacro (robot description, xacro)
@@ -1,53 +1,29 @@
 <?xml version='1.0'?>
-<robot name="ezrassor" xmlns:xacro="http://www.ros.org/wiki/xacro">
+<robot name="ezrassor"
+    xmlns:xacro="http://www.ros.org/wiki/xacro">
     <!-- Inertia Tensors Used: https://en.wikipedia.org/wiki/List_of_moments_of_inertia#List_of_3D_inertia_tensors -->
     <xacro:macro name="cylinder_inertia" params="m r h">
-    <inertia
-        ixx="${m*((3*r*r)+(h*h))/12}" ixy = "0"                 ixz = "0"
-                                  iyy="${m*((3*r*r)+(h*h))/12}" iyz = "0"
-                                                            izz="${(m*(r*r))/2}"
-    />
+        <inertia ixx="${m*((3*r*r)+(h*h))/12}" ixy = "0"                 ixz = "0" iyy="${m*((3*r*r)+(h*h))/12}" iyz = "0" izz="${(m*(r*r))/2}" />
     </xacro:macro>
     <xacro:macro name="box_inertia" params="m x y z">
-    <inertia  ixx="${m*(y*y+z*z)/12}" ixy = "0" ixz = "0"
-        iyy="${m*(x*x+z*z)/12}" iyz = "0"
-        izz="${m*(x*x+z*z)/12}"
-    />
+        <inertia ixx="${m*(y*y+z*z)/12}" ixy = "0" ixz = "0" iyy="${m*(x*x+z*z)/12}" iyz = "0" izz="${m*(x*x+z*z)/12}" />
     </xacro:macro>
     <xacro:macro name="sphere_inertia" params="m r">
-    <inertia  ixx="${2*m*r*r/5}" ixy = "0" ixz = "0"
-        iyy="${2*m*r*r/5}" iyz = "0"
-        izz="${2*m*r*r/5}"
-    />
+        <inertia ixx="${2*m*r*r/5}" ixy = "0" ixz = "0" iyy="${2*m*r*r/5}" iyz = "0" izz="${2*m*r*r/5}" />
     </xacro:macro>
     <xacro:macro name="slender_rod_along_y_inertia" params="m l mass_about">
         <xacro:if value="${mass_about == 'end'}">
-            <inertia
-                ixx="${1/3*m*(l*l)}" ixy = "0"
+            <inertia ixx="${1/3*m*(l*l)}" ixy = "0"
                 ixz = "0" iyy="0"
                 iyz = "0" izz="${1/3*m*(l*l)}" />
         </xacro:if>
         <xacro:unless value="${mass_about == 'center'}">
-            <inertia
-                ixx="${1/12*m*(l*l)}" ixy = "0"
+            <inertia ixx="${1/12*m*(l*l)}" ixy = "0"
                 ixz = "0" iyy="0"
                 iyz = "0" izz="${1/12*m*(l*l)}" />
         </xacro:unless>
     </xacro:macro>
-    <!-- VISUAL AND COLLISION MACROS -->
-    <xacro:macro name="robot_arm">
-        <mesh filename="package://ezrassor_sim_description/meshes/drum_arm_short.dae" scale="1.0 1.0 1.0"></mesh>
-    </xacro:macro>
-    <xacro:macro name="robot_arm_drum">
-        <mesh filename="package://ezrassor_sim_description/meshes/drum.dae" scale="0.35 0.35 0.35"></mesh>
-    </xacro:macro>
-    <xacro:macro name="robot_wheel">
-        <mesh filename="package://ezrassor_sim_description/meshes/wheel.dae" scale="0.35 0.35 0.35"></mesh>
-    </xacro:macro>
     <xacro:macro name="base_unit">
-        <mesh filename="package://ezrassor_sim_description/meshes/base_unit.dae" scale="0.35 0.35 0.35"></mesh>
-    </xacro:macro>
-    <xacro:macro name="drum_arm">
-        <mesh filename="package://ezrassor_sim_description/meshes/drum_arm.dae" scale="0.35 0.35 0.35"></mesh>
+        <mesh filename="file://$(find ezrassor_sim_description)/meshes/base_unit.dae" scale="0.35 0.35 0.35"></mesh>
     </xacro:macro>
 </robot>
