Commit message: Added depthimg to laserscan node, improved obstacle detection, and changed tf frames

File: urdf/ezrassor.xacro.urdf (robot description, URDF)
Before this commit: robot ezrassor, 2 links, 1 joints
Links:
- added link camera_depth_frame
- added link camera_link, mass 0.1; collision box size=0.01 0.01 0.01; visual box size=0.01 0.01 0.01
Joints:
- added joint camera_depth_joint: type fixed, parent camera_link, child camera_depth_frame, origin xyz=0 0 0 rpy=${-pi/2} 0 ${-pi/2}
- added joint camera_joint: type fixed, parent base_link, child camera_link, origin xyz=.3 0 -.1 rpy=0 0 0, axis 0 1 0
